File: basestation-board-v2/basestation.brd (EAGLE design)
At the start: 73.4 x 45.5 mm, 68 parts, among them IC1 STM32F072, IC2 MCP1700TT, IC3 MCP73831, IC4 MCP1700TT, J1 SWD_SHROUD_SMD, Q1 BSS84, Q2 BSS84, SW1 ROTARTY_ENCODER, U1 NHD-C0216CIZ-FSW, U2 RFM98, U3 RN4020, X1 BU-SMA-V, X2 CRYSTAL-GROUNDED, X3 BN35N61, X4 MINI-USB-32005-301

Commit message: improvments
Parts:
- removed JP1: USB_MICROB_PLUGCONN-11752, SparkFun-Connectors:USB-B-MICRO-SMD_V03
- removed LED5, LED6: (no value), led:CHIP-LED0805
- removed SJ1, SJ2: (no value), jumper:SJ
- removed U$2: (no value), Mine:SUSF-XSM
- added C18: (no value), passives-7351:C0603-N
- added JP3: USB-MICRO, Mine:MOLEX_47589-0001
- added U$3: JST-ZR-2SMD, Mine:JST-ZR-2-SMD
- LED3, LED4: device led:LED3MM -> dtb:LED3MM
- X4: value MINI-USB-32005-301 -> 1-227161-6; device con-cypressindustries:32005-301 -> con-coax:AMP_227161
- moved X4 16.9 mm to (-48.3, -3.05)
- moved D1 3.24 mm to (62.4, 30.7), turned to 0 degrees
- moved Q2 0.51 mm to (62.4, 27.9)
Connections:
- removed net N$19: IC1.35, SJ1.2
- removed net N$20: IC1.36, SJ2.2
- net +3V3: now also C18.2, IC1.36; no longer SJ2.1
- net DM: now also JP3.D-; no longer JP1.D-1
- net DP: now also JP3.D+; no longer JP1.D+1
- net GND: now also C18.1, IC1.35, JP3.GND, U$3.2; no longer JP1.GND1, LED5.C, LED6.C, SJ1.1
- net LED2: now also IC1.42; no longer IC1.3
- net N$10: now also RN2.6; no longer RN2.7
- net N$16: no longer LED6.A
- net N$17: no longer LED5.A
- net N$28: now also JP3.ID; no longer JP1.ID1
- net N$33: now also U$3.1
- net N$35: now also JP3.VCC; no longer JP1.VBUS1
- net N$6: now also RN2.7; no longer RN2.6
- net SW1: now also IC1.3; no longer IC1.42
Routing:
- net N$26: track 0.00 -> 42.8 mm, vias 0 -> 4
- net ROT_A: track 15.9 -> 33.5 mm, vias 0 -> 2
- net LED2: track 13.6 -> 28.8 mm
- net +3V3: track 191.4 -> 206.1 mm, vias 6 -> 8
- net ROT_M: track 5.23 -> 16.3 mm, vias 1 -> 2
- net VBUS: track 44.0 -> 37.5 mm, vias 5 -> 2
- net GND: track 203.3 -> 209.3 mm, vias 144 -> 152
- net R_INT: track 103.8 -> 109.3 mm
- net SW1: track 26.4 -> 21.0 mm, vias 0 -> 1
- net VIN_S: track 68.3 -> 65.0 mm, vias 3 -> 4
- net VBAT_S: track 38.6 -> 37.2 mm
- net N$6: track 15.2 -> 16.5 mm
- net N$17: track 10.6 -> 9.93 mm
- net N$33: track 45.6 -> 46.2 mm
- net DP: track 13.3 -> 13.9 mm
- added copper zone on layer 16, net N$18
Other:
- outline, holes or cut-outs redrawn
- board text removed: "BT ON"
- board text removed: "DATA"
