File: basestation-board-v2/basestation.sch (EAGLE design)
At the start: 67 parts, among them IC1 STM32F072, IC2 MCP1700TT, IC3 MCP73831, IC4 MCP1700TT, J1 SWD_SHROUD_SMD, Q1 BSS84, Q2 BSS84, SW1 ROTARTY_ENCODER, U1 NHD-C0216CIZ-FSW, U2 RFM98, U3 RN4020, X1 BU-SMA-V, X2 CRYSTAL-GROUNDED, X3 BN35N61, X4 MINI-USB-32005-301

Commit message: improvments
Parts:
- removed JP1: USB_MICROB_PLUGCONN-11752, SparkFun-Connectors:USB_MICROB_PLUGCONN-11752
- removed LED5, LED6: (no value), led:LEDCHIP-LED0805
- removed SJ1, SJ2: (no value), jumper:SJ
- added C18: (no value), passives-7351:CAPACITOR0603-N
- added JP3: USB-MICRO, Mine:USB-MICRO
- added U$3: JST-ZR-2SMD, Mine:JST-ZR-2SMD
- LED3, LED4: device led:LED3MM -> dtb:LED3MM
- X4: value MINI-USB-32005-301 -> 1-227161-6; device con-cypressindustries:MINI-USB-32005-301 -> con-coax:1-227161-6
Connections:
- removed net N$19: IC1.VSS1, SJ1.2
- removed net N$20: IC1.VDDIO, SJ2.2
- net +3V3: now also C18.2, IC1.VDDIO; no longer SJ2.1
- net DM: now also JP3.D-; no longer JP1.D-
- net DP: now also JP3.D+; no longer JP1.D+
- net GND: now also C18.1, IC1.VSS1, JP3.GND, U$3.2; no longer JP1.GND, LED5.C, LED6.C, SJ1.1
- net LED2: now also IC1.PB6; no longer IC1.PC14
- net N$10: now also RN2C.2; no longer RN2B.2
- net N$16: no longer LED6.A
- net N$17: no longer LED5.A
- net N$28: now also JP3.ID; no longer JP1.ID
- net N$33: now also U$3.1
- net N$35: now also JP3.VCC; no longer JP1.VCC
- net N$6: now also RN2B.2; no longer RN2C.2
- net SW1: now also IC1.PC14; no longer IC1.PB6
Other:
- note added: "TODO"
- note added: "improve power arrangment?"
- note added: "test bi-colour led"
- moved on the sheet: RN2B, RN2C
